Commit message: [update] huge update

File: assets/keyboards/simplified/12996/mobility_merged.urdf (robot description, URDF)
Before this commit: robot full108keyboard, 106 links, 105 joints
Links:
- link link_0: geometry visual mesh filename=/home/chengjing/Desktop/keyboard_typer/assets/keyboards/sim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

Commit message: update

File: assets/keyboards/simplified/12996/mobility_merged.urdf (robot description, URDF)
Before this commit: robot full108keyboard, 106 links, 105 joints
Links:
- link link_0: geometry visual mesh filename=textured_objs/original-106.obj
- link link_1: geometry collision mesh filename=merged_collision_meshes/merged_link_1.stl; visual mesh filename=textured_objs/original-287.obj
- link link_10: geometry collision mesh filename=merged_collision_meshes/merged_link_10.stl; visual mesh filename=textured_objs/original-146.obj
- link link_100: geometry collision mesh filename=merged_collision_meshes/merged_link_100.stl; visual mesh filename=textured_objs/original-264.obj
- link link_101: geometry collision mesh filename=merged_collision_meshes/merged_link_101.stl; visual mesh filename=textured_objs/original-263.obj
- link link_102: geometry collision mesh filename=merged_collision_meshes/merged_link_102.stl; visual mesh filename=textured_objs/original-262.obj
- link link_103: geometry collision mesh filename=merged_collision_meshes/merged_link_103.stl; visual mesh filename=textured_objs/original-100.obj
- link link_104: geometry collision mesh filename=merged_collision_meshes/merged_link_104.stl; visual mesh filename=textured_objs/original-274.obj
- link link_11: geometry collision mesh filename=merged_collision_meshes/merged_link_11.stl; visual mesh filename=textured_objs/original-284.obj
- link link_12: geometry collision mesh filename=merged_collision_meshes/merged_link_12.stl; visual mesh filename=textured_objs/original-18.obj
- link link_13: geometry collision mesh filename=merged_collision_meshes/merged_link_13.stl; visual mesh filename=textured_objs/original-131.obj
- link link_14: geometry collision mesh filename=merged_collision_meshes/merged_link_14.stl; visual mesh filename=textured_objs/original-127.obj
- link link_15: geometry collision mesh filename=merged_collision_meshes/merged_link_15.stl; visual mesh filename=textured_objs/original-138.obj
- link link_16: geometry collision mesh filename=merged_collision_meshes/merged_link_16.stl; visual mesh filename=textured_objs/original-126.obj
- link link_17: geometry collision mesh filename=merged_collision_meshes/merged_link_17.stl; visual mesh filename=textured_objs/original-10.obj
- link link_18: geometry collision mesh filename=merged_collision_meshes/merged_link_18.stl; visual mesh filename=textured_objs/original-229.obj
- link link_19: geometry collision mesh filename=merged_collision_meshes/merged_link_19.stl; visual mesh filename=textured_objs/original-22.obj
- link link_2: geometry collision mesh filename=merged_collision_meshes/merged_link_2.stl; visual mesh filename=textured_objs/original-205.obj
- link link_20: geometry collision mesh filename=merged_collision_meshes/merged_link_20.stl; visual mesh filename=textured_objs/original-305.obj
- link link_21: geometry collision mesh filename=merged_collision_meshes/merged_link_21.stl; visual mesh filename=textured_objs/original-299.obj
- link link_22: geometry collision mesh filename=merged_collision_meshes/merged_link_22.stl; visual mesh filename=textured_objs/original-113.obj
- link link_23: geometry collision mesh filename=merged_collision_meshes/merged_link_23.stl; visual mesh filename=textured_objs/original-231.obj
- link link_24: geometry collision mesh filename=merged_collision_meshes/merged_link_24.stl; visual mesh filename=textured_objs/original-21.obj
- link link_25: geometry collision mesh filename=merged_collision_meshes/merged_link_25.stl; visual mesh filename=textured_objs/original-233.obj
- link link_26: geometry collision mesh filename=merged_collision_meshes/merged_link_26.stl; visual mesh filename=textured_objs/original-234.obj
- link link_27: geometry collision mesh filename=merged_collision_meshes/merged_link_27.stl; visual mesh filename=textured_objs/original-108.obj
- link link_28: geometry collision mesh filename=merged_collision_meshes/merged_link_28.stl; visual mesh filename=textured_objs/original-17.obj
- link link_29: geometry collision mesh filename=merged_collision_meshes/merged_link_29.stl; visual mesh filename=textured_objs/original-280.obj
- link link_3: geometry collision mesh filename=merged_collision_meshes/merged_link_3.stl; visual mesh filename=textured_objs/original-207.obj
- link link_30: geometry collision mesh filename=merged_collision_meshes/merged_link_30.stl; visual mesh filename=textured_objs/original-26.obj
- link link_31: geometry collision mesh filename=merged_collision_meshes/merged_link_31.stl; visual mesh filename=textured_objs/original-112.obj
- link link_32: geometry collision mesh filename=merged_collision_meshes/merged_link_32.stl; visual mesh filename=textured_objs/original-122.obj
- link link_33: geometry collision mesh filename=merged_collision_meshes/merged_link_33.stl; visual mesh filename=textured_objs/original-119.obj
- link link_34: geometry collision mesh filename=merged_collision_meshes/merged_link_34.stl; visual mesh filename=textured_objs/original-118.obj
- link link_35: geometry collision mesh filename=merged_collision_meshes/merged_link_35.stl; visual mesh filename=textured_objs/original-109.obj
- link link_36: geometry collision mesh filename=merged_collision_meshes/merged_link_36.stl; visual mesh filename=textured_objs/original-254.obj
- link link_37: geometry collision mesh filename=merged_collision_meshes/merged_link_37.stl; visual mesh filename=textured_objs/original-271.obj
- link link_38: geometry collision mesh filename=merged_collision_meshes/merged_link_38.stl; visual mesh filename=textured_objs/original-272.obj
- link link_39: geometry collision mesh filename=merged_collision_meshes/merged_link_39.stl; visual mesh filename=textured_objs/original-19.obj
- link link_4: geometry collision mesh filename=merged_collision_meshes/merged_link_4.stl; visual mesh filename=textured_objs/original-209.obj
- link link_40: geometry collision mesh filename=merged_collision_meshes/merged_link_40.stl; visual mesh filename=textured_objs/original-277.obj
- link link_41: geometry collision mesh filename=merged_collision_meshes/merged_link_41.stl; visual mesh filename=textured_objs/original-278.obj
- link link_42: geometry collision mesh filename=merged_collision_meshes/merged_link_42.stl; visual mesh filename=textured_objs/original-252.obj
- link link_43: geometry collision mesh filename=merged_collision_meshes/merged_link_43.stl; visual mesh filename=textured_objs/original-251.obj
- link link_44: geometry collision mesh filename=merged_collision_meshes/merged_link_44.stl; visual mesh filename=textured_objs/original-250.obj
- link link_45: geometry collision mesh filename=merged_collision_meshes/merged_link_45.stl; visual mesh filename=textured_objs/original-249.obj
- link link_46: geometry collision mesh filename=merged_collision_meshes/merged_link_46.stl; visual mesh filename=textured_objs/original-15.obj
- link link_47: geometry collision mesh filename=merged_collision_meshes/merged_link_47.stl; visual mesh filename=textured_objs/original-247.obj
- link link_48: geometry collision mesh filename=merged_collision_meshes/merged_link_48.stl; visual mesh filename=textured_objs/original-246.obj
- link link_49: geometry collision mesh filename=merged_collision_meshes/merged_link_49.stl; visual mesh filename=textured_objs/original-123.obj
- link link_5: geometry collision mesh filename=merged_collision_meshes/merged_link_5.stl; visual mesh filename=textured_objs/original-211.obj
- link link_50: geometry collision mesh filename=merged_collision_meshes/merged_link_50.stl; visual mesh filename=textured_objs/original-235.obj
- link link_51: geometry collision mesh filename=merged_collision_meshes/merged_link_51.stl; visual mesh filename=textured_objs/original-121.obj
- link link_52: geometry collision mesh filename=merged_collision_meshes/merged_link_52.stl; visual mesh filename=textured_objs/original-116.obj
- link link_53: geometry collision mesh filename=merged_collision_meshes/merged_link_53.stl; visual mesh filename=textured_objs/original-236.obj
- link link_54: geometry collision mesh filename=merged_collision_meshes/merged_link_54.stl; visual mesh filename=textured_objs/original-110.obj
- link link_55: geometry collision mesh filename=merged_collision_meshes/merged_link_55.stl; visual mesh filename=textured_objs/original-245.obj
- link link_56: geometry collision mesh filename=merged_collision_meshes/merged_link_56.stl; visual mesh filename=textured_objs/original-111.obj
- link link_57: geometry collision mesh filename=merged_collision_meshes/merged_link_57.stl; visual mesh filename=textured_objs/original-165.obj
- link link_58: geometry collision mesh filename=merged_collision_meshes/merged_link_58.stl; visual mesh filename=textured_objs/original-102.obj
- link link_59: geometry collision mesh filename=merged_collision_meshes/merged_link_59.stl; visual mesh filename=textured_objs/original-244.obj
- link link_6: geometry collision mesh filename=merged_collision_meshes/merged_link_6.stl; visual mesh filename=textured_objs/original-20.obj
- link link_60: geometry collision mesh filename=merged_collision_meshes/merged_link_60.stl; visual mesh filename=textured_objs/original-243.obj
- link link_61: geometry collision mesh filename=merged_collision_meshes/merged_link_61.stl; visual mesh filename=textured_objs/original-242.obj
- link link_62: geometry collision mesh filename=merged_collision_meshes/merged_link_62.stl; visual mesh filename=textured_objs/original-241.obj
- link link_63: geometry collision mesh filename=merged_collision_meshes/merged_link_63.stl; visual mesh filename=textured_objs/original-16.obj
- link link_64: geometry collision mesh filename=merged_collision_meshes/merged_link_64.stl; visual mesh filename=textured_objs/original-239.obj
- link link_65: geometry collision mesh filename=merged_collision_meshes/merged_link_65.stl; visual mesh filename=textured_objs/original-238.obj
- link link_66: geometry collision mesh filename=merged_collision_meshes/merged_link_66.stl; visual mesh filename=textured_objs/original-276.obj
- link link_67: geometry collision mesh filename=merged_collision_meshes/merged_link_67.stl; visual mesh filename=textured_objs/original-275.obj
- link link_68: geometry collision mesh filename=merged_collision_meshes/merged_link_68.stl; visual mesh filename=textured_objs/original-152.obj
- link link_69: geometry collision mesh filename=merged_collision_meshes/merged_link_69.stl; visual mesh filename=textured_objs/original-156.obj
- link link_7: geometry collision mesh filename=merged_collision_meshes/merged_link_7.stl; visual mesh filename=textured_objs/original-290.obj
- link link_70: geometry collision mesh filename=merged_collision_meshes/merged_link_70.stl; visual mesh filename=textured_objs/original-158.obj
- link link_71: geometry collision mesh filename=merged_collision_meshes/merged_link_71.stl; visual mesh filename=textured_objs/original-101.obj
- link link_72: geometry collision mesh filename=merged_collision_meshes/merged_link_72.stl; visual mesh filename=textured_objs/original-273.obj
- link link_73: geometry collision mesh filename=merged_collision_meshes/merged_link_73.stl; visual mesh filename=textured_objs/original-162.obj
- link link_74: geometry collision mesh filename=merged_collision_meshes/merged_link_74.stl; visual mesh filename=textured_objs/original-95.obj
- link link_75: geometry collision mesh filename=merged_collision_meshes/merged_link_75.stl; visual mesh filename=textured_objs/original-172.obj
- link link_76: geometry collision mesh filename=merged_collision_meshes/merged_link_76.stl; visual mesh filename=textured_objs/original-168.obj
- link link_77: geometry collision mesh filename=merged_collision_meshes/merged_link_77.stl; visual mesh filename=textured_objs/original-182.obj
- link link_78: geometry collision mesh filename=merged_collision_meshes/merged_link_78.stl; visual mesh filename=textured_objs/original-190.obj
- link link_79: geometry collision mesh filename=merged_collision_meshes/merged_link_79.stl; visual mesh filename=textured_objs/original-237.obj
- link link_8: geometry collision mesh filename=merged_collision_meshes/merged_link_8.stl; visual mesh filename=textured_objs/original-292.obj
- link link_80: geometry collision mesh filename=merged_collision_meshes/merged_link_80.stl; visual mesh filename=textured_objs/original-270.obj
- link link_81: geometry collision mesh filename=merged_collision_meshes/merged_link_81.stl; visual mesh filename=textured_objs/original-295.obj
- link link_82: geometry collision mesh filename=merged_collision_meshes/merged_link_82.stl; visual mesh filename=textured_objs/original-141.obj
- link link_83: geometry collision mesh filename=merged_collision_meshes/merged_link_83.stl; visual mesh filename=textured_objs/original-319.obj
- link link_84: geometry collision mesh filename=merged_collision_meshes/merged_link_84.stl; visual mesh filename=textured_objs/original-269.obj
- link link_85: geometry collision mesh filename=merged_collision_meshes/merged_link_85.stl; visual mesh filename=textured_objs/original-268.obj
- link link_86: geometry collision mesh filename=merged_collision_meshes/merged_link_86.stl; visual mesh filename=textured_objs/original-105.obj
- link link_87: geometry collision mesh filename=merged_collision_meshes/merged_link_87.stl; visual mesh filename=textured_objs/original-12.obj
- link link_88: geometry collision mesh filename=merged_collision_meshes/merged_link_88.stl; visual mesh filename=textured_objs/original-217.obj
- link link_89: geometry collision mesh filename=merged_collision_meshes/merged_link_89.stl; visual mesh filename=textured_objs/original-11.obj
- link link_9: geometry collision mesh filename=merged_collision_meshes/merged_link_9.stl; visual mesh filename=textured_objs/original-145.obj
- link link_90: geometry collision mesh filename=merged_collision_meshes/merged_link_90.stl; visual mesh filename=textured_objs/original-221.obj
- link link_91: geometry collision mesh filename=merged_collision_meshes/merged_link_91.stl; visual mesh filename=textured_objs/original-220.obj
- link link_92: geometry collision mesh filename=merged_collision_meshes/merged_link_92.stl; visual mesh filename=textured_objs/original-13.obj
- link link_93: geometry collision mesh filename=merged_collision_meshes/merged_link_93.stl; visual mesh filename=textured_objs/original-224.obj
- link link_94: geometry collision mesh filename=merged_collision_meshes/merged_link_94.stl; visual mesh filename=textured_objs/original-223.obj
- link link_95: geometry collision mesh filename=merged_collision_meshes/merged_link_95.stl; visual mesh filename=textured_objs/original-222.obj
- link link_96: geometry collision mesh filename=merged_collision_meshes/merged_link_96.stl; visual mesh filename=textured_objs/original-103.obj
- link link_97: geometry collision mesh filename=merged_collision_meshes/merged_link_97.stl; visual mesh filename=textured_objs/original-266.obj
- link link_98: geometry collision mesh filename=merged_collision_meshes/merged_link_98.stl; visual mesh filename=textured_objs/original-104.obj
- link link_99: geometry collision mesh filename=merged_collision_meshes/merged_link_99.stl; visual mesh filename=textured_objs/original-265.obj

Commit message: add base collision back for reaslistic simulation, retain code for pressing test

File: assets/keyboards/simplified/12996/mobility_merged.urdf (robot description, URDF)
Before this commit: robot full108keyboard, 106 links, 105 joints
Links:
- link link_0: geometry collision mesh filename=merged_collision_meshes/merged_link_0.stl; visual mesh filename=textured_objs/original-106.obj
